File: MotorControl/Boards/motorControl.brd (EAGLE design)
At the start: 80 x 76.2 mm, 67 parts, among them IC101 STM32F103C8T6, IC201 LM2596S-5V, IC202 LM1117-3V3, IC301 MCP2561-E/SN, IC302 RS485SOIC, IC303 RS485SOIC, IC304 RS485SOIC, IC305 RS485SOIC, IC401 MIC5014YM, IC403 IPB160, J501 POWER_IN_COCK_OUT_24V, J502 PROG, J503 PANEL_SIGNAL, J504 OPTRONIK, J505 TRIGGER, J506 COCK_DRIVER, J507 MTR_AZ_CTRL, J508 MTR_EL_CTRL, Q101 8MHz, Q401 A03401, Q402 2N2222A

Commit message: v2.1.0
Parts:
- removed C301: 100n, rcl:C0603
- removed D301, D502, D503, D504: SCHOTTKY, diode:MICROMELF-W
- removed IC403: IPB160, infineon:PG-TO263-7
- removed L103: GREEN, led:CHIP-LED0805
- removed Q402: 2N2222A, scorpion:SOT23
- removed R405: 100k, rcl:R0603
- removed R503, R504, R505: 10k, resistor:R0603
- removed R506, R507: 100R, resistor:R0603
- removed SJ102: (no value), SparkFun:SJ_2S-TRACE
- removed SJ201, SJ202: SOLDERJUMPERTRACE, SparkFun:SJ_2S-TRACE
- added C501: 100n, resistor:C0603
- added D401: SS34, adafruit:SMADIODE
- added IC402: PC817, optocoupler:DIL04
- added J509: COCK_DRIVER, SparkFun-Connectors:XH-6-VERT-SMD
- added KK401: (no value), heatsink:BV_240X170-HOLE
- added L102: GREEN, led:CHIP-LED0805
- added R1, R2, R3, R4: 120R, resistor:R0603
- added SJ101: (no value), SparkFun:SJ_2S-TRACE
- C101: value 100n -> 10n
- D402: value SS34 -> 10V; device adafruit:SMADIODE -> encPhone:DO-4148
- IC401: value MIC5014YM -> PC817; device microchip:SO-08 -> optocoupler:DIL04
- J501: value POWER_IN_COCK_OUT_24V -> PROG; device con-ptr500:AK300/8 -> SparkFun-Connectors:XH-4-VERT-SMD
- J502: value PROG -> BUS; device SparkFun-Connectors:XH-4-VERT-SMD -> SparkFun-Connectors:XH-8-VERT-SMD
- J503: value PANEL_SIGNAL -> OPTRONIK
- J504: value OPTRONIK -> MTR_AZ_COMM; device SparkFun-Connectors:XH-8-VERT-SMD -> SparkFun-Connectors:XH-4-VERT-SMD
- J505: value TRIGGER -> MTR_EL_COMM; device con-ptr500:AK300/2 -> SparkFun-Connectors:XH-4-VERT-SMD
- J506: value COCK_DRIVER -> LIMIT_SWITCH
- J507: value MTR_AZ_CTRL -> POWER_IN; device SparkFun-Connectors:XH-6-VERT-SMD -> con-ptr500:AK300/2
- J508: value MTR_EL_CTRL -> TRIGGER_OUT; device SparkFun-Connectors:XH-6-VERT-SMD -> con-ptr500:AK300/2
- Q401: value A03401 -> IRF9530; device scorpion:SOT23 -> transistor-power:TO220BV
- R401: value 100k -> 470R
- R403: value 100k -> 330R
- R501, R502: value 100R -> 120R
- moved J508 66.0 mm to (6.35, 22.2), turned to 90 degrees
- moved J507 62.8 mm to (6.35, 12.1), turned to 90 degrees
- moved IC201 58.5 mm to (50.2, 66.7), turned to 270 degrees
- moved U$1 57.5 mm to (64.3, 65.8), flipped to the top, turned to 90 degrees
- moved C202 56.0 mm to (59.1, 53.3)
- moved D402 54.1 mm to (12.1, 35.6), turned to 90 degrees
- moved D501 51.5 mm to (48.9, 28.3)
- moved R302 51.4 mm to (78.7, 62.2), turned to 270 degrees
- moved R401 48.6 mm to (11.4, 36.8), flipped to the bottom, turned to 180 degrees
- moved J503 48.5 mm to (10.2, 54.3)
- moved R303 46.7 mm to (78.7, 57.1), turned to 270 degrees
- moved IC302 46.6 mm to (73.7, 62.2), turned to 270 degrees
- moved J501 46.0 mm to (64.1, 33.0), turned to 270 degrees
- moved J505 44.4 mm to (85.1, 44.5), turned to 270 degrees
- moved C104 43.2 mm to (59.1, 10.2), flipped to the top, turned to 90 degrees
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Connections:
- net N$58 renamed VBAT
- removed net GATE: IC401.5, IC403.1, R401.2
- removed net MTR_AZ_ZERO: IC101.11, R506.1
- removed net MTR_EL_ZERO: IC101.20, R507.2
- removed net N$29: IC101.27
- removed net N$32: Q402.1, R404.1, R405.2
- removed net N$33: IC101.17
- removed net N$34: J508.5, R507.1
- removed net N$35: J506.4, R502.1
- removed net N$36: J507.5, R506.2
- removed net N$5 (its old number): IC101.19, R103.1
- removed net N$8: Q401.1, Q402.3, R403.1
- removed net TRIGGER_+: D402.C, IC401.3, IC403.2, IC403.3, IC403.5, IC403.6, IC403.7, J505.2, R401.1
- removed net TRIGGER_INPUT: IC401.2, Q401.3, R402.2
- removed net TRIGGER_START: J503.3, R404.2
- removed net VIDEO_DAY_CAM: J503.5, J504.4
- removed net VIDEO_GND: J503.6, J504.3
- removed net VIDEO_THERMAL_CAM: J503.4, J504.5
- new net +12V: C201.+, IC201.1, J502.1, J503.6
- new net BUS_RESV: J502.8
- new net BUS_TRIGGER_PULSE: J502.7, R403.2
- new net BUS_VIDEO+: J502.5, J503.2
- new net BUS_VIDEO-: J502.6, J503.1
- new net LIM_AZ: IC101.17, J506.2
- new net LIM_EL_DOWN: IC101.19, J506.6
- new net LIM_EL_UP: IC101.18, J506.4
- new net N$12: IC101.16
- new net N$22: J509.6, R501.1
- new net N$24: C501.2, J509.4, R2.1
- new net N$42: D402.C, Q401.G, R401.2
- new net N$43: IC401.3, IC402.4, R402.2
- new net N$44: IC401.1, R403.1
- new net N$45: IC402.1, R404.1
- new net N$47: D402.A, IC401.4
- new net TRIGGER+: D401.C, J508.2, Q401.D
- net +24V: now also J507.1, Q401.S, R401.1, R402.1; no longer C201.+, IC201.1, IC401.1, IC403.4, J501.1, J501.2, J501.3, J501.4, J504.1
- net +3V3: now also D501.C; no longer Q401.2, R403.2
- net +5V: no longer C301.1, R503.1, R504.1, R505.1
- net AGND: now also J501.4, L102.C, SJ101.1; no longer L103.C, SJ102.1
- net BUS_CANH: now also J502.3, J503.4; no longer J503.2, J504.7
- net BUS_CANL: now also J502.4, J503.3; no longer J503.1, J504.8
- net BUS_RXD: now also R1.1; no longer D301.A
- net COCK_ALM: now also R4.2; no longer R502.2
- net COCK_AWO: now also R502.2; no longer D502.C
- net COCK_DIR: now also R2.2; no longer D504.C
- net COCK_PLS: now also R3.2; no longer D503.C
- net COCK_POS: now also IC101.27; no longer IC101.18
- net GND: now also C201.-, C202.-, D201.A, IC201.3, IC201.5, IC201.6, IC401.2, IC402.2, J502.2, J503.5, J506.1, J506.3, J506.5, J509.1, SJ101.2; no longer C301.2, IC401.4, J502.4, J506.6, J507.6, J508.6, R402.1, R405.1, SJ102.2, SJ201.1, SJ202.1
- net MTR_AZ_RX_A: now also J504.4; no longer J507.4
- net MTR_AZ_RX_B: now also J504.3; no longer J507.3
- net MTR_AZ_TX_A: now also J504.2; no longer J507.2
- net MTR_AZ_TX_B: now also J504.1; no longer J507.1
- net MTR_EL_RX_A: now also J505.4; no longer J508.4
- net MTR_EL_RX_B: now also J505.3; no longer J508.3
- net MTR_EL_TX_A: now also J505.2; no longer J508.2
- net MTR_EL_TX_B: now also J505.1; no longer J508.1
- net N$10: now also R1.2; no longer D301.C
- net N$13: now also J509.5, R502.1; no longer J506.5, R501.1
- net N$2: now also L102.A; no longer L103.A
- net N$25: now also J509.3, R3.1; no longer D504.A, J506.1, R505.2
- net N$26: now also J509.2, R4.1; no longer D503.A, J506.2, R504.2
- net N$27: now also J501.1; no longer J502.1
- net N$28: now also IC101.20; no longer D502.A, J506.3, R503.2
- net N$3: now also R103.1
- net RST: now also C501.1
- net SWCLK: now also J501.3; no longer J502.3
- net SWDIO: now also J501.2; no longer J502.2
- net TRIGGER_ENABLE: now also IC101.11, R404.2; no longer IC101.16, Q402.2
- net V-: now also D401.A, IC402.3, J507.2, J508.1; no longer C201.-, C202.-, D201.A, D402.A, IC201.3, IC201.5, IC201.6, J501.5, J501.6, J501.7, J501.8, J504.2, J505.1, SJ201.2, SJ202.2
- net VDD: no longer D501.C
Routing:
- net GND: track 13.6 -> 316.3 mm, vias 2 -> 4
- net BUS_CANL: track 22.5 -> 153.3 mm
- net BUS_CANH: track 31.8 -> 151.7 mm
- net LIM_AZ: track 0.00 -> 74.7 mm
- net +5V: track 152.7 -> 82.5 mm
- net LIM_EL_UP: track 0.00 -> 66.5 mm
- net LIM_EL_DOWN: track 0.00 -> 57.5 mm
- net N$24: track 0.00 -> 49.1 mm, vias 0 -> 2
- net BUS_TRIGGER_PULSE: track 0.00 -> 48.8 mm
- net +12V: track 0.00 -> 44.8 mm
- net COCK_DIR: track 59.2 -> 15.7 mm, vias 1 -> 0
- net TRIGGER_ENABLE: track 13.8 -> 55.1 mm, vias 1 -> 0
- net COCK_PLS: track 58.9 -> 18.6 mm, vias 1 -> 0
- net GATE: track 40.1 -> 0.00 mm, vias 2 -> 0
- net COCK_AWO: track 52.8 -> 12.9 mm, vias 1 -> 0
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- added copper zone on layer 16, net AGND
- added copper zone on layer 1, net VDD
- removed copper zone on layer 1, net +24V
- removed copper zone on layer 16, net +24V
- removed copper zone on layer 1, net +5V
- removed copper zone on layer 1, net AGND
- removed copper zone on layer 1, net LM2596_OUT
- removed copper zone on layer 1, net TRIGGER_+
- removed copper zone on layer 16, net TRIGGER_+
- removed copper zone on layer 1, net V-
- removed copper zone on layer 16, net V-
- removed copper zone on layer 16, net VDD
Other:
- board size 80 x 76.2 mm -> 94 x 76.2 mm
- board text added: "GND"
- board text added: "USART1_RX"
- board text added: "USART1_TX"
- board text added: "motorControl_RCWS 20190826"
- board text removed: "PT. Respati Solusi Rekatama"
- board text removed: "RCWS - motorControl_v2.0.0"
