File: Optronik/Boards/Optronik.sch (EAGLE design)
At the start: 113 parts, among them IC101 STM32F103C8T6, IC201 LM2596S-5V, IC202 LM2596S-ADJ, IC301 STM32F103C8T6, IC401 RS485SOIC, IC402 L293DD, IC403 MCP2561-E/SN, IC404 MCP2561-E/SN, IC405 MAX232SOIC16, IC406 RS485SOIC, J501 PANEL, J502 SONY, J503 THERMAL_DALI_VIDEO, J504 THERMAL_DALI_MOTOR, J505 LRF_NOPTEL, J506 IMU, J507 GPS, J508 MCU_CAM_PROG, J509 MCU_MAIN_PROG, Q101 8MHz, Q201 A03401, T401 1N2222A, T402 1N2222A

Commit message: v2.1.0
Parts:
- removed C206, C210: 470u/35V, resistor:CPOL-EU153CLV-1012
- removed C211: 10n, rcl:C-EUC0603
- removed C212: 1000u/6V3, resistor:CPOL-EU153CLV-0810
- removed C307, C411, C412, C501, C502, C503, C504, C505: 100n, resistor:C-EUC0603
- removed C405: 100n, rcl:C-EUC0603
- removed C406, C407, C408, C409, C410: 1u, resistor:C-EUC0603
- removed D202, D501: SS34, adafruit:DIODESMA
- removed D301, D502, D503: SCHOTTKY, diode:DIODE-MICROMELF-W
- removed F501, F502, F503, F504, F505: 500mA, rcl:L-EUL0805
- removed IC203: (no value), SparkFun:V_REG_LM1117SOT223
- removed IC401, IC406: RS485SOIC, SparkFun-DigitalIC:RS485SOIC
- removed IC402: L293DD, adafruit:L293DD
- removed IC403, IC404: MCP2561-E/SN, microchip:MCP2561-E/SN
- removed IC405: MAX232SOIC16, SparkFun-DigitalIC:MAX232SOIC16
- removed J202: (no value), SparkFun-Connectors:M02-XH-VERT-SMD
- removed J501: PANEL, SparkFun-Connectors:M08-XH-RA
- removed J502: SONY, SparkFun-Connectors:M06-XH-RA
- removed J503: THERMAL_DALI_VIDEO, SparkFun-Connectors:M06-XH-RA
- removed J504: THERMAL_DALI_MOTOR, SparkFun-Connectors:M08-XH-RA
- removed J505: LRF_NOPTEL, SparkFun-Connectors:M06-XH-RA
- removed J506: IMU, SparkFun-Connectors:M04-XH-RA
- removed J507: GPS, SparkFun-Connectors:M04-XH-RA
- removed J508: MCU_CAM_PROG, SparkFun-Connectors:M04-XH-VERT
- removed J509: MCU_MAIN_PROG, SparkFun-Connectors:M04-XH-VERT
- removed L202: 33uH, scorpion:PA4342
- removed L301, L302, L401: FB_0603, rc-master:FB_0603
- removed R201A, R201B: 120R, resistor:R-EU_R0603
- removed R202A, R202B, R408: 1k, resistor:R-EU_R0603
- removed R406, R407, R410, R411, R504, R505: 100R, resistor:R-EU_R0603
- removed R409, R414, R415, R416, R417: 100R, rcl:R-EU_R0603
- removed R412, R413: 100, resistor:R-EU_R0603
- removed R501, R502: 1R, resistor:R-EU_0411/3V
- removed R503: 10k, resistor:R-EU_R0603
- removed R506: 120R, rcl:R-EU_R0603
- removed SJ1: SOLDERJUMPERTRACE, SparkFun-Passives:SOLDERJUMPERTRACE
- removed SJ201, SJ202: SOLDERJUMPERTRACE, SparkFun:SOLDERJUMPERTRACE
- removed T401, T402: 1N2222A, SparkFun-DiscreteSemi:TRANSISTOR_NPNSOT23
- added C108, C302, C303, C401, C402, C403: 100n, resistor:C-EUC0603
- added C109: 2u2, resistor:C-EUC0603
- added C203: 1000u/6V3, resistor:CPOL-EU153CLV-0810
- added D402: SCHOTTKY, diode:DIODE-MICROMELF-W
- added F401, F402, F403, F404: 500mA, rcl:L-EUL0805
- added IC302: MCP2561-E/SN, microchip:MCP2561-E/SN
- added IC303: MAX2021, SparkFun-DigitalIC:MAX232SOIC16
- added IC304: TS5V330CDR, Texas Instruments_By_element14_Batch_1:TS5V330CDR
- added J401: PANEL, SparkFun-Connectors:M06-XH-RA
- added J402: SONY, SparkFun-Connectors:M06-XH-RA
- added J403: THERMAL_DALI_VIDEO, SparkFun-Connectors:M06-XH-RA
- added J404: LRF_NOPTEL, SparkFun-Connectors:M06-XH-RA
- added J405: IMU, SparkFun-Connectors:M04-XH-RA
- added J406: PROG_DEBUG, SparkFun-Connectors:M06-XH-VERT
- added L103: GREEN, led:LEDCHIP-LED0805
- added Q202: 2N2222, scorpion:2N2222-REFLOW
- added R103: 1k, resistor:R-EU_R0603
- added R303, R304, R305, R306, R307: 120R, rcl:R-EU_R0603
- added R401: 10k, resistor:R-EU_R0603
- added R402: 120R, resistor:R-EU_R0603
- C101: value 100n -> 10n
- C202: value 1000u/6V3 -> 470u/35V; device resistor:CPOL-EU153CLV-0810 -> resistor:CPOL-EU153CLV-1012
- C301: device resistor:C-EUC0603 -> rcl:C-EUC0603
- C404: device rcl:C-EUC0603 -> resistor:C-EUC0603
- D401: value SCHOTTKY -> SS34; device diode:DIODE-MICROMELF-W -> adafruit:DIODESMA
- IC101: value STM32F103C8T6 -> STM32F446RET6; device ST Microelctronics_By_element14_Batch_1:STM32F103C8T6 -> micro-stm_v3:STM32F401RBT; LINK https://www.tokopedia.com/embedded-world/stm32-stm32f103c8t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 -> (none)
- IC202: value LM2596S-ADJ -> LM1117-3V3; device ON Semiconductor_By_element14_Batch_1:LM2596S-ADJ -> SparkFun:V_REG_LM1117SOT223
- IC301: value STM32F103C8T6 -> RS485SOIC; device ST Microelctronics_By_element14_Batch_1:STM32F103C8T6 -> SparkFun-DigitalIC:RS485SOIC; LINK https://www.tokopedia.com/embedded-world/stm32-stm32f103c8t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 -> (none)
- J201: value (none) -> JP_5V
- R204, R403, R404: value 100R -> 120R
- R301: value 100K -> 120R; device resistor:R-EU_R0603 -> rcl:R-EU_R0603
- R302: value 100K -> 120R; device resistor:R-EU_R0603 -> rcl:R-EU_R0603; DNP (none) -> T
- R405: value 1k -> 120R
- SJ101: device SparkFun-Passives:SOLDERJUMPERTRACE -> SparkFun:SOLDERJUMPERTRACE; BOM (none) -> EXCLUDE; DNP (none) -> T
Connections:
- removed net +24V: C201.+, C206.+, D501.C, IC201.VIN, IC202.VIN
- removed net AGND1: C301.2, C304.1, C305.1, C306.1, C307.1, IC301.VSSA, IC301.VSS_1, IC301.VSS_2, IC301.VSS_3, J508.1, R301.2, SJ1.1
- removed net BOOT0: IC101.BOOT0, R101.1
- removed net BUS1_RXD: IC101.PA11/USART1_CTS/CAN_RX/USB_DM/TIM1_CH4, R415.2
- removed net BUS1_TXD: IC101.PA12/USART1_RTS/CAN_TX/USB_DP/TIM1_ETR, R414.2
- removed net BUS2_RXD: IC301.PB8/TIM4_CH3[I2C1_SCL/CAN_RX], R417.2
- removed net BUS2_TXD: IC301.PB9/TIM4_CH4[I2C1_SDA/CAN_TX], R416.2
- removed net FEED1: C211.2, IC202.FB, R201A.2, R202B.2
- removed net GPS_A_TX: IC406.A, J507.4, R412.2
- removed net GPS_B_RX: IC406.B, J507.3, R413.1
- removed net GPS_RTS: IC101.PB14/SPI2_MISO/USART3_RTS/TIM1_CH2N, IC406.DE
- removed net GPS_RXD: IC101.PB10/I2C2_SCL/USART3_TX[TIM2_CH3], IC406.DI, R413.2
- removed net GPS_TXD: IC101.PB11/I2C2_SDA/USART3_RX[TIM2_CH4], IC406.RO, R412.1
- removed net LRF_EN: IC101.PC13/TAMPERRTC, J505.6, R503.2
- removed net MCO: IC101.PA8/USART1_CK/TIM1_CH1/MCO, IC301.PD0/OSC_IN
- removed net N$10: IC101.PB2/BOOT1
- removed net N$11: IC101.PC14/OSC32_IN
- removed net N$15: D501.A, J501.2
- removed net N$16: D202.C, IC202.VOUT, L202.1
- removed net N$19: IC101.PB0/ADC12_IN8/TIM3_CH3[TIM1_CH2N]
- removed net N$25: IC101.PA5/SPI1_SCK/ADC12_IN5
- removed net N$26: IC101.PA4/SPI1_NSS/USART2_CK/ADC12_IN4
- removed net N$27: IC101.PB12/SPI2_NSS/I2C2_SMBAL/USART3_CK/TIM1_BKIN
- removed net N$28: IC101.PB13/SPI2_SCK/USART3_CTS/TIM1_CH1N
- removed net N$35: F503.1, J504.1
- removed net N$36: IC301.PA6/SPI1_MISO/ADC12_IN6/TIM3_CH1[TIM1_BKIN]
- removed net N$37: IC301.PC15/OSC32_OUT
- removed net N$41: D502.A, J509.4
- removed net N$46: IC301.PA3/USART2_RX/ADC12_IN3/TIM2_CH4
- removed net N$52: C503.2, F501.2, J502.5
- removed net N$54: IC101.PA0/WKUP/USART2_CTS/ADC12_IN0/TIM2_CH1_ETR
- removed net N$57: IC101.PC15/OSC32_OUT
- removed net N$63: C210.+, C211.1, J202.2, L202.2, R202A.2
- removed net N$66: IC301.PA7/SPI1_MOSI/ADC12_IN7/TIM3_CH2[TIM1_CH1N]
- removed net N$71: IC404.TXD, R416.1
- removed net N$76: IC301.PB0/ADC12_IN8/TIM3_CH3[TIM1_CH2N]
- removed net N$77: IC402.1-2EN, R403.2
- removed net N$78: IC402.3-4EN, R406.1
- removed net N$79: IC301.PB1/ADC12_IN9/TIM3_CH4[TIM1_CH3N]
- removed net N$80: D503.A, J508.4
- removed net N$89: R405.1, T401.B
- removed net N$90: IC402.2A, T401.C
- removed net N$91: IC402.4A, T402.C
- removed net N$92: R408.2, T402.B
- removed net RST1: C301.1, D301.A, IC301.NRST, R302.2
- removed net SWCLK1: IC101.JTCK/SWCLK[PA14], J509.2
- removed net SWCLK2: IC301.JTCK/SWCLK[PA14], J508.2
- removed net SWDIO1: IC101.JTMS/SWDIO[PA13], J509.3
- removed net SWDIO2: IC301.JTMS/SWDIO[PA13], J508.3
- removed net THERMAL_ADC_FOCUS: IC301.PA4/SPI1_NSS/USART2_CK/ADC12_IN4, R411.2
- removed net THERMAL_ADC_ZOOM: IC301.PA5/SPI1_SCK/ADC12_IN5, R410.2
- removed net THERMAL_A_TX: IC401.A, J503.3
- removed net THERMAL_B_RX: IC401.B, J503.4
- removed net THERMAL_FB_FOCUS: C412.2, J504.3, R411.1, R501.1
- removed net THERMAL_FB_ZOOM: C411.2, J504.4, R410.1, R502.2
- removed net THERMAL_RTS: IC301.PA12/USART1_RTS/CAN_TX/USB_DP/TIM1_ETR, IC401.DE
- removed net TH_FOCUS+: IC402.3Y, J504.7
- removed net TH_FOCUS-: IC402.4Y, J504.8
- removed net TH_FOCUS_DIR: IC301.PB5/I2C1_SMBAL[TIM3_CH2/SPI1_MOSI], R407.2, R408.1
- removed net TH_FOCUS_PLS: IC301.JNTRST[PB4/TIM3_CH1/SPI1_MISO], R406.2
- removed net TH_ZOOM+: IC402.1Y, J504.5
- removed net TH_ZOOM-: IC402.2Y, J504.6
- removed net TH_ZOOM_DIR: IC301.JTDO[PB3/TIM2_CH2/TRACESWO/SPI1_CLK], R404.1, R405.2
- removed net TH_ZOOM_PLS: IC301.JTDI[PA15/TIM2_CH1_ETR/SPI1_NSS], R403.1
- removed net V-: C201.-, C202.-, C206.-, C210.-, D201.A, D202.A, IC201.EN, IC201.GND, IC202.EN, IC202.GND, J501.1, R201B.1, SJ201.2, SJ202.2
- removed net VDD1: C304.2, C305.2, C306.2, D301.C, D503.C, IC301.VDD_1, IC301.VDD_2, IC301.VDD_3, IC401.VCC, L301.1, L302.1, R302.1
- removed net VDDA1: C307.2, IC301.VDDA, L302.2
- removed net VIDEO-: J501.8, J502.1, J503.1
- new net !LRF_EN: IC101MCU.PC15, J404.6, R401.2
- new net BUS_RXD: IC101MCU.PA11, R304.2
- new net BUS_TXD: IC101MCU.PA12, R303.2
- new net CAM_SELECT: IC101MCU.PB15, R307.2
- new net DEBUG_RXD: IC101MCU.PA0-WKUP, J406.3
- new net DEBUG_TXD: IC101MCU.PA1, J406.2
- new net LED: IC101MCU.PB6, R103.1
- new net SONY_VDD: C401.2, F401.2, J402.5
- new net TCK: IC101MCU.PA14, J406.4
- new net THERMAL_A: IC301.A, J403.3, R301.1
- new net THERMAL_B: IC301.B, J403.4, R301.2
- new net THERMAL_DE: IC101MCU.PB3, IC301.DE
- new net TMS: IC101MCU.PA13, J406.5
- new net USART1_RXD: IC101MCU.PA10
- new net USART1_TXD: IC101MCU.PA9
- new net VBAT: IC101MCU.VBAT
- new net VIDEO_GND: J401.1, J402.1, J403.1
- new net VIDEO_OUT: IC304.DA, J401.2
- net +12V: now also C201.+, D401.C, F401.1, IC201.VIN; no longer F501.1, J202.1
- net +3V3: now also C203.+, IC202.OUT, IC202.OUT@1, IC301.VCC, R401.1; no longer C212.+, IC203.OUT, IC203.OUT@1, IC406.VCC, L301.2
- net +5V: now also C301.1, C302.1, C305.2, F403.2, F404.2, IC202.IN, IC302.VCC, IC303.VCC, IC304.VCC; no longer C404.1, C405.1, C406.1, C407.2, C505.1, F503.2, F504.2, F505.2, IC203.IN, IC402.VDD, IC403.VCC, IC404.VCC, IC405.VCC, J507.2, L401.1
- net AGND: now also C108.1, C109.1, IC101MCU.VSSA, IC101PWR.VSS@1, IC101PWR.VSS@2, IC101PWR.VSS@3, IC101PWR.VSS@4; no longer IC101.VSSA, IC101.VSS_1, IC101.VSS_2, IC101.VSS_3
- net BOOT1: now also IC101MCU.BOOT0, R101.1; no longer IC301.BOOT0, R301.1
- net BUS_CANH: now also IC302.CAN_H, J401.4, R302.2; no longer IC403.CAN_H, IC404.CAN_H, J501.3, R506.1
- net BUS_CANL: now also IC302.CAN_L, J401.3, R302.1; no longer IC403.CAN_L, IC404.CAN_L, J501.4, R506.2
- net GND: now also C201.-, C202.-, C203.-, C301.2, C302.2, C306.1, C401.1, C402.2, C403.2, D201.A, IC201.EN, IC201.GND, IC202.ADJ, IC301./RE, IC301.GND, IC302.GND, IC302.STBY, IC303.GND, IC304.GND, IC304.~EN, J401.5, J402.6, J403.6, J404.1, J405.1, J406.1, L103.C, Q202.E; no longer C212.-, C405.2, C406.2, C408.1, C411.1, C412.1, C501.2, C502.2, C503.1, C504.2, C505.2, IC203.ADJ, IC401./RE, IC401.GND, IC402.GND, IC402.GND@1, IC402.GND@2, IC402.GND@3, IC402.GND@4, IC402.GND@5, IC402.GND@6, IC402.GND@7, IC403.GND, IC403.STBY, IC404.GND, IC404.STBY, IC405.GND, IC406./RE, IC406.GND, J502.6, J503.6, J504.2, J505.1, J506.1, J507.1, J509.1, R501.2, R502.1, SJ1.2, SJ201.1, SJ202.1, T401.E, T402.E
- net IMU_RX: now also IC303.T2OUT, J405.3; no longer IC405.T2OUT, J506.3
- net IMU_RXD: now also IC101MCU.PC12, R305.2; no longer IC101.PA2/USART2_TX/ADC12_IN2/TIM2_CH3, R409.2
- net IMU_TX: now also IC303.R2IN, J405.4; no longer IC405.R2IN, J506.4
- net IMU_TXD: now also IC101MCU.PD2, R306.2; no longer D401.A, IC101.PA3/USART2_RX/ADC12_IN3/TIM2_CH4
- net LRF_RXD: now also IC101MCU.PA2, R402.2; no longer IC101.PA9/USART1_TX/TIM1_CH2, R504.2
- net LRF_TXD: now also IC101MCU.PA3, R403.2; no longer IC101.PA10/USART1_RX/TIM1_CH3, R505.2
- net N$1: now also D402.A, J406.6; no longer IC301.PA9/USART1_TX/TIM1_CH2
- net N$12: now also D401.A, J401.6; no longer IC101.PB1/ADC12_IN9/TIM3_CH4[TIM1_CH3N]
- net N$13: now also IC101MCU.PC9; no longer IC101.PB6/I2C1_SCL/TIM4_CH1[USART1_TX]
- net N$14: now also IC101MCU.PC8; no longer IC101.PB7/I2C1_SDA/TIM4_CH2[USART1_RX]
- net N$17: now also Q202.B, R204.1; no longer R201A.1, R201B.2
- net N$18: now also IC302.RXD, R304.1; no longer R202A.1, R202B.1
- net N$2: now also C102.1, IC101MCU.OSC_IN, Q101.2; no longer IC101.PB8/TIM4_CH3[I2C1_SCL/CAN_RX]
- net N$20: now also IC101MCU.PA8; no longer IC101.JTDI[PA15/TIM2_CH1_ETR/SPI1_NSS]
- net N$21: now also IC101MCU.PB9; no longer IC301.PB14/SPI2_MISO/USART3_RTS/TIM1_CH2N
- net N$22: now also L103.A, R103.2; no longer IC402.VCC, L401.2
- net N$23: now also IC101MCU.PA5; no longer IC101.PA7/SPI1_MOSI/ADC12_IN7/TIM3_CH2[TIM1_CH1N]
- net N$24: now also C103.2, IC101MCU.OSC_OUT, Q101.1; no longer IC301.PC13/TAMPERRTC
- net N$3: now also J402.3, R404.1; no longer IC301.PD1/OSC_OUT
- net N$30: now also IC101MCU.PA7; no longer IC101.PB15/SPI2_MOSI/TIM1_CH3N
- net N$31: now also C306.2, IC303.V-; no longer C408.2, IC405.V-
- net N$32: now also C303.2, IC303.C1+; no longer C409.2, IC405.C1+
- net N$33: now also C304.2, IC303.C2+; no longer C410.2, IC405.C2+
- net N$34: now also IC101MCU.PA4; no longer IC101.JTDO[PB3/TIM2_CH2/TRACESWO/SPI1_CLK]
- net N$38: now also IC101MCU.PB0; no longer IC301.VBAT
- net N$39: now also Q202.C; no longer R204.1
- net N$4: now also C109.2, IC101MCU.VCAP1; no longer IC101.JNTRST[PB4/TIM3_CH1/SPI1_MISO]
- net N$40: now also IC101MCU.PB1; no longer IC301.PA0/WKUP/USART2_CTS/ADC12_IN0/TIM2_CH1_ETR
- net N$42: now also IC101MCU.PB2; no longer IC101.PA6/SPI1_MISO/ADC12_IN6/TIM3_CH1[TIM1_BKIN]
- net N$43: now also IC101MCU.PB10; no longer IC402.3A, R407.1
- net N$44: now also IC101MCU.PB12; no longer IC301.PA1/USART2_RTS/ADC12_IN1/TIM2_CH2
- net N$45: now also IC101MCU.PB13; no longer IC301.PA2/USART2_TX/ADC12_IN2/TIM2_CH3
- net N$47: now also C402.1, F402.1, J403.5; no longer C501.1, F502.1, J503.5
- net N$48: now also C403.1, F403.1, J404.2; no longer C502.1, F504.1, J505.2
- net N$49: now also IC302.TXD, R303.1; no longer IC403.TXD, R414.1
- net N$50: now also IC101MCU.PC5; no longer IC402.1A, R404.2
- net N$51: now also IC101MCU.PB14; no longer IC101.PB5/I2C1_SMBAL[TIM3_CH2/SPI1_MOSI]
- net N$53: now also IC101MCU.PC4; no longer IC101.PA1/USART2_RTS/ADC12_IN1/TIM2_CH2
- net N$55: now also C404.1, F404.1, J405.2; no longer C504.1, F505.1, J506.2
- net N$56: now also J404.3, R403.1; no longer J505.3, R505.1
- net N$58: now also IC101MCU.PC3; no longer IC101.VBAT
- net N$59: now also J404.4, R402.1; no longer J505.4, R504.1
- net N$6: now also IC101MCU.PA6; no longer C103.2, IC101.PD1/OSC_OUT, Q101.1
- net N$60: now also IC101MCU.PC2; no longer IC301.PC14/OSC32_IN
- net N$61: now also IC101MCU.PC1; no longer IC301.PB12/SPI2_NSS/I2C2_SMBAL/USART3_CK/TIM1_BKIN
- net N$62: now also IC101MCU.PC0; no longer IC301.PB13/SPI2_SCK/USART3_CTS/TIM1_CH1N
- net N$64: now also IC101MCU.PB8; no longer IC301.PB15/SPI2_MOSI/TIM1_CH3N
- net N$65: now also IC101MCU.PB7; no longer IC301.PA8/USART1_CK/TIM1_CH1/MCO
- net N$67: now also IC101MCU.PB5; no longer IC403.RXD, R415.1
- net N$68: now also C303.1, IC303.C1-; no longer C409.1, IC405.C1-
- net N$69: now also C304.1, IC303.C2-; no longer C410.1, IC405.C2-
- net N$7: now also IC101MCU.PC14; no longer C102.1, IC101.PD0/OSC_IN, Q101.2
- net N$70: now also IC101MCU.PB4; no longer IC301.PB2/BOOT1
- net N$72: now also C305.1, IC303.V+; no longer C407.1, IC405.V+
- net N$73: now also IC304.IN, R307.1; no longer IC404.RXD, R417.1
- net N$74: now also IC303.T2IN, R305.1; no longer IC405.T2IN, R409.1
- net N$75: now also IC303.R2OUT, R306.1; no longer D401.C, IC405.R2OUT
- net N$8: now also IC101MCU.PC13; no longer IC101.PB9/TIM4_CH4[I2C1_SDA/CAN_TX]
- net N$9: now also J402.4, R405.1; no longer IC301.PA10/USART1_RX/TIM1_CH3
- net RST: now also IC101MCU.NRST; no longer IC101.NRST
- net SONY_RXD: now also IC101MCU.PC6, R404.2; no longer IC301.PB10/I2C2_SCL/USART3_TX[TIM2_CH3], J502.3
- net SONY_TXD: now also IC101MCU.PC7, R405.2; no longer IC301.PB11/I2C2_SDA/USART3_RX[TIM2_CH4], J502.4
- net THERMAL_PWR_EN: now also IC101MCU.PA15; no longer IC301.PA11/USART1_CTS/CAN_RX/USB_DM/TIM1_CH4
- net THERMAL_RXD: now also IC101MCU.PC10, IC301.DI; no longer IC301.PB6/I2C1_SCL/TIM4_CH1[USART1_TX], IC401.DI
- net THERMAL_TXD: now also IC101MCU.PC11, IC301.RO; no longer IC301.PB7/I2C1_SDA/TIM4_CH2[USART1_RX], IC401.RO
- net THERMAL_VDD: now also F402.2; no longer F502.2
- net VDD: now also C108.2, D402.C, IC101MCU.VDDA, IC101PWR.VDD@1, IC101PWR.VDD@2, IC101PWR.VDD@3, IC101PWR.VDD@4; no longer D502.C, IC101.VDDA, IC101.VDD_1, IC101.VDD_2, IC101.VDD_3, R503.1
- net VIDEO_SONY+: now also IC304.S1A, J402.2; no longer J501.7, J502.2
- net VIDEO_THERMAL+: now also IC304.S2A, J403.2; no longer J501.6, J503.2
Other:
- note added: "BUS"
- note added: "IMU & GPS"
- note removed: "COMM"
- note removed: "MOTORIZED ZOMM & FOCUS"
- note removed: "Vout = 1.23(1 + (R_ATAS)/(R_BAWAH) ) 240R <= R_BAWAH <= 1k5"
