File: Panel/Boards/panel446.sch (EAGLE design)
At the start: 61 parts, among them IC101 STM32F103C8T6, IC201 LM2596S-5V, IC202 LM1117-3V3, IC301 MCP2561-E/SN, IC302 RS485SOIC, IC303 RS485SOIC, IC304 RS485SOIC, IC305 RS485SOIC, IC401 PC817, IC402 PC817, J501 PROG, J502 BUS, J503 OPTRONIK, J504 MTR_AZ_COMM, J505 MTR_EL_COMM, J506 LIMIT_SWITCH, J507 POWER_IN, J508 TRIGGER_OUT, J509 COCK_DRIVER, Q101 8MHz, Q401 IRF9530

Commit message: v2.1.0
Parts:
- removed C201: 470u/35V, resistor:CPOL-EU153CLV-1012
- removed C204: 1000u/6V3, resistor:CPOL-EU153CLV-0810
- removed C501: 100n, resistor:C-EUC0603
- removed D201: SS34, adafruit:DIODESMA
- removed D501: SCHOTTKY, diode:DIODE-MICROMELF-W
- removed IC401, IC402: PC817, optocoupler:PC817
- removed J501: PROG, SparkFun-Connectors:M04-XH-VERT-SMD
- removed J502: BUS, SparkFun-Connectors:M08-XH-VERT-SMD
- removed J503: OPTRONIK, SparkFun-Connectors:M06-XH-VERT-SMD
- removed J504: MTR_AZ_COMM, SparkFun-Connectors:M04-XH-VERT-SMD
- removed J505: MTR_EL_COMM, SparkFun-Connectors:M04-XH-VERT-SMD
- removed J506: LIMIT_SWITCH, SparkFun-Connectors:M06-XH-VERT-SMD
- removed J507: POWER_IN, con-ptr500:AK300/2
- removed J508: TRIGGER_OUT, con-ptr500:AK300/2
- removed J509: COCK_DRIVER, SparkFun-Connectors:M06-XH-VERT-SMD
- removed KK401: (no value), heatsink:TO220T25-HOLE
- removed L102: GREEN, led:LEDCHIP-LED0805
- removed L201: 33uH, scorpion:PA4342
- removed Q401: IRF9530, transistor-power:IRF9530
- removed R1, R2, R3, R4, R501, R502: 120R, resistor:R-EU_R0603
- removed R403, R404: 330R, rcl:R-EU_R0603
- added C108, C301, C401, C402: 100n, resistor:C-EUC0603
- added C109: 2u2, rcl:C-EUC0805
- added F402: 500mA, rcl:L-EUL0805
- added IC203: LM1117-3V3, SparkFun:V_REG_LM1117SOT223
- added IC306: ESP01, esp8266modules:ESP01
- added J401: BUS, SparkFun-Connectors:M08-XH-VERT
- added J402: BUTTON, SparkFun-Connectors:M08-XH-VERT
- added J403: POWER, SparkFun-Connectors:M04-XH-VERT
- added J404: DC CONVERTER, SparkFun-Connectors:M04-XH-VERT
- added J405: PROG, SparkFun-Connectors:M04-XH-VERT
- added J406: DEBUG, SparkFun-Connectors:M04-XH-VERT
- added J407: GPS, SparkFun-Connectors:M04-XH-VERT
- added J408: PWR_MONITOR, SparkFun-Connectors:M02-XH-RA
- added J409: PC, SparkFun-Connectors:M06-XH-VERT
- added J410: SIGHTLINE, SparkFun-Connectors:M06-XH-VERT
- added L103: GREEN, led:LEDCHIP-LED0805
- added R201: 1k, rcl:R-EU_R0603
- added R202: 100k, rcl:R-EU_R0603
- added R306: 330R, rcl:R-EU_R0603
- added R307, R308, R405, R406: 120R, rcl:R-EU_R0603
- D401: value SS34 -> SCHOTTKY; device adafruit:DIODESMA -> diode:DIODE-MICROMELF-W
- D402: value 10V -> SCHOTTKY; device encPhone:ZENER -> diode:DIODE-MICROMELF-W
- IC101: value STM32F103C8T6 -> STM32F446RET6; device ST Microelctronics_By_element14_Batch_1:STM32F103C8T6 -> micro-stm_v3:STM32F401RBT; LINK https://www.tokopedia.com/embedded-world/stm32-stm32f103c8t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 -> (none)
- IC201: value LM2596S-5V -> MIC5014YM; device ON Semiconductor_By_element14_Batch_1:LM2596S-ADJ -> microchip:MIC5014YM
- IC202: value LM1117-3V3 -> IPB160; device SparkFun:V_REG_LM1117SOT223 -> infineon:IPB160
- IC302, IC303, IC304: value RS485SOIC -> PC817-DIL; device SparkFun-DigitalIC:RS485SOIC -> optocoupler:PC817-DIL
- IC305: value RS485SOIC -> MAX485DIL; device SparkFun-DigitalIC:RS485SOIC -> SparkFun:MAX485DIL
- R301, R304: device resistor:R-EU_R0603 -> rcl:R-EU_R0603; DNP (none) -> T
- R302, R303: device resistor:R-EU_R0603 -> rcl:R-EU_R0603
- R305: value 120R -> 330R; device resistor:R-EU_R0603 -> rcl:R-EU_R0603; DNP (none) -> T
- R401: value 470R -> 10k
- R402: value 100k -> 1k
- SJ101: BOM (none) -> EXCLUDE; DNP (none) -> T
Connections:
- removed net +24V: J507-1.KL, Q401.S, R401.1, R402.1
- removed net BOOT0: IC101.BOOT0, R101.1
- removed net COCK_ALM: IC101.PA10/USART1_RX/TIM1_CH3, R4.2
- removed net COCK_AWO: IC101.PB15/SPI2_MOSI/TIM1_CH3N, R502.2
- removed net COCK_DIR: IC101.PA8/USART1_CK/TIM1_CH1/MCO, R2.2
- removed net COCK_PLS: IC101.PA9/USART1_TX/TIM1_CH2, R3.2
- removed net COCK_POS: IC101.PB14/SPI2_MISO/USART3_RTS/TIM1_CH2N, R501.2
- removed net LIM_AZ: IC101.PA7/SPI1_MOSI/ADC12_IN7/TIM3_CH2[TIM1_CH1N], J506.2
- removed net LIM_EL_DOWN: IC101.PB1/ADC12_IN9/TIM3_CH4[TIM1_CH3N], J506.6
- removed net LIM_EL_UP: IC101.PB0/ADC12_IN8/TIM3_CH3[TIM1_CH2N], J506.4
- removed net LM2596_OUT: D201.C, IC201.VOUT, L201.1
- removed net MTR_AZ_RXD: IC101.PA3/USART2_RX/ADC12_IN3/TIM2_CH4, IC302.RO
- removed net MTR_AZ_RX_A: IC303.A, J504.4, R303.2
- removed net MTR_AZ_RX_B: IC303.B, J504.3, R303.1
- removed net MTR_AZ_TXD: IC101.PA2/USART2_TX/ADC12_IN2/TIM2_CH3, IC303.DI
- removed net MTR_AZ_TX_A: IC302.A, J504.2, R302.2
- removed net MTR_AZ_TX_B: IC302.B, J504.1, R302.1
- removed net MTR_EL_RXD: IC101.PB11/I2C2_SDA/USART3_RX[TIM2_CH4], IC304.RO
- removed net MTR_EL_RX_A: IC305.A, J505.4, R305.2
- removed net MTR_EL_RX_B: IC305.B, J505.3, R305.1
- removed net MTR_EL_TXD: IC101.PB10/I2C2_SCL/USART3_TX[TIM2_CH3], IC305.DI
- removed net MTR_EL_TX_A: IC304.A, J505.2, R304.2
- removed net MTR_EL_TX_B: IC304.B, J505.1, R304.1
- removed net N$10: IC301.RXD, R1.2
- removed net N$12: IC101.PA6/SPI1_MISO/ADC12_IN6/TIM3_CH1[TIM1_BKIN]
- removed net N$13: J509.5, R502.1
- removed net N$14: IC101.PB9/TIM4_CH4[I2C1_SDA/CAN_TX]
- removed net N$15: IC101.PB8/TIM4_CH3[I2C1_SCL/CAN_RX]
- removed net N$21: IC101.PA4/SPI1_NSS/USART2_CK/ADC12_IN4
- removed net N$22: J509.6, R501.1
- removed net N$27: D501.A, J501.1
- removed net N$47: D402.A, IC401.COL
- removed net RST: C101.1, C501.1, D101.A, IC101.NRST, R102.2
- removed net SWCLK: IC101.JTCK/SWCLK[PA14], J501.3
- removed net SWDIO: IC101.JTMS/SWDIO[PA13], J501.2
- removed net TRIGGER+: D401.C, J508-2.KL, Q401.D
- removed net TRIGGER_ENABLE: IC101.PA1/USART2_RTS/ADC12_IN1/TIM2_CH2, R404.2
- removed net V-: D401.A, IC402.EMIT, J507-2.KL, J508-1.KL
- new net !RST: C101.1, C402.1, D101.A, IC101MCU.NRST, R102.2
- new net BATT_VOLT: C401.1, IC101MCU.PA7, R401.1, R402.2
- new net BOOT1: IC101MCU.BOOT0, R101.1
- new net BUTTON_RXD: IC101MCU.PB10, J402.7
- new net BUTTON_TXD: IC101MCU.PC5, J402.6
- new net DEBUG_RXD: IC101MCU.PA2, J406.3
- new net DEBUG_TXD: IC101MCU.PA3, J406.2
- new net GATE: IC201.GATE, IC202.G, R202.2
- new net GPS_A_RX: IC305.A, J407.3
- new net GPS_B_TX: IC305.B, J407.4
- new net GPS_RXD: IC101MCU.PC6, R308.2
- new net GPS_TXD: IC101MCU.PC7, R307.2
- new net N$29: IC101MCU.PA8
- new net N$31: C102.1, IC101MCU.OSC_IN, Q101.2
- new net N$33: IC101MCU.PA5
- new net N$34: IC101MCU.PA4
- new net N$38: IC101MCU.PB13
- new net N$39: IC101MCU.PB7
- new net N$40: IC101MCU.PB6
- new net N$41: IC101MCU.PB3
- new net N$46: IC301.RXD, R303.1
- new net N$49: IC301.TXD, R302.1
- new net N$50: IC302.A, R304.1
- new net N$56: IC101MCU.PA1
- new net N$58: IC303.A, R305.1
- new net N$59: IC305.RO, R307.1
- new net N$60: IC305.DI, R308.1
- new net N$61: C402.2, J406.4
- new net N$65: F402.1, J410.1
- new net N$68: IC304.A, R306.1
- new net N$69: IC201.INPUT, R201.1
- new net N$8: J409.4, J410.4, R406.1
- new net PC_IGNITE: IC304.COL, J409.6
- new net PC_IGNITION: IC101MCU.PC9, R306.2
- new net PC_PWR_CHECK: J409.5, R305.2
- new net PC_PWR_CHECK_IN: IC101MCU.PC8, IC303.COL
- new net PWR_BATT+: IC201.V+, IC202.D, J402.1, J403.1, R401.2
- new net PWR_FROM_EMER: J402.2, R201.2
- new net PWR_RESV: J403.4
- new net PWR_TO_CONVERTER: IC201.SOURCE, IC202.S, J404.1, R202.1
- new net TCK: IC101MCU.PA14, J405.2
- new net TMS: IC101MCU.PA13, J405.3
- new net TRACKER_RXD: IC101MCU.PA9, R405.2
- new net TRACKER_TXD: IC101MCU.PA10, R406.2
- new net TRIGGER_IN: IC101MCU.PB12, J402.3
- new net TRIG_PULSE_OUT: IC101MCU.PB15, R304.2
- new net WIFI_EN: IC101MCU.PA15, IC306.CH_PD
- new net WIFI_RST: C301.1, IC101MCU.PC12
- new net WIFI_RXD: IC101MCU.PC10, IC306.RXD
- new net WIFI_TXD: IC101MCU.PC11, IC306.TXD
- net +12V: now also D401.C, IC302.COL, J401.1, J402.4, J403.3, J404.2, J408.1, J409.1; no longer C201.+, IC201.VIN, J502.1, J503.6
- net +3V3: now also C202.+, IC203.OUT, IC203.OUT@1, J402.5; no longer C204.+, D501.C, IC202.OUT, IC202.OUT@1, IC302.VCC, IC303./RE, IC303.DE, IC303.VCC, IC304.VCC, IC305./RE, IC305.DE, IC305.VCC
- net +5V: now also F402.2, IC203.IN, IC305.VCC, J404.3, J407.2; no longer C202.+, IC201.FB, IC202.IN, L201.2
- net AGND: now also C108.1, C109.1, IC101MCU.VSSA, IC101PWR.VSS@1, IC101PWR.VSS@2, IC101PWR.VSS@3, IC101PWR.VSS@4, IC306.GND, J405.1, J406.1, L103.C; no longer IC101.VSSA, IC101.VSS_1, IC101.VSS_2, IC101.VSS_3, J501.4, L102.C
- net BUS_CANH: now also J401.3, R301.2; no longer J502.3, J503.4
- net BUS_CANL: now also J401.4, R301.1; no longer J502.4, J503.3
- net BUS_RESV: now also J401.8; no longer J502.8
- net BUS_RXD: now also IC101MCU.PA11, R303.2; no longer IC101.PA11/USART1_CTS/CAN_RX/USB_DM/TIM1_CH4, R1.1
- net BUS_TRIGGER_PULSE: now also IC302.EMIT, J401.7; no longer J502.7, R403.2
- net BUS_TXD: now also IC101MCU.PA12, R302.2; no longer IC101.PA12/USART1_RTS/CAN_TX/USB_DP/TIM1_ETR, R301.1
- net BUS_VIDEO+: now also J401.5, J410.6; no longer J502.5, J503.2
- net BUS_VIDEO-: now also J401.6, J410.5; no longer J502.6, J503.1
- net GND: now also C401.2, D401.A, IC203.ADJ, IC302.C, IC303.C, IC303.EMIT, IC304.C, IC304.EMIT, IC305.DE, IC305.RE, J401.2, J402.8, J403.2, J404.4, J407.1, J408.2, J409.2, J410.2, R402.1; no longer C201.-, C204.-, D201.A, IC201.EN, IC202.ADJ, IC302./RE, IC302.DE, IC302.GND, IC303.GND, IC304./RE, IC304.DE, IC304.GND, IC401.C, IC402.C, J502.2, J503.5, J506.1, J506.3, J506.5, J509.1
- net N$1: now also IC101MCU.PB9; no longer IC101.PB12/SPI2_NSS/I2C2_SMBAL/USART3_CK/TIM1_BKIN
- net N$11: now also IC101MCU.PB8; no longer IC101.PC14/OSC32_IN
- net N$16: now also IC101MCU.PC4; no longer IC101.PB7/I2C1_SDA/TIM4_CH2[USART1_RX]
- net N$17: now also IC101MCU.PC3; no longer IC101.JTDO[PB3/TIM2_CH2/TRACESWO/SPI1_CLK]
- net N$18: now also IC101MCU.PC2; no longer IC101.JNTRST[PB4/TIM3_CH1/SPI1_MISO]
- net N$19: now also IC101MCU.PD2, R103.1; no longer IC101.PB6/I2C1_SCL/TIM4_CH1[USART1_TX]
- net N$2: now also C109.2, IC101MCU.VCAP1; no longer L102.A, R103.2
- net N$20: now also L103.A, R103.2; no longer IC101.JTDI[PA15/TIM2_CH1_ETR/SPI1_NSS]
- net N$23: now also IC101MCU.PB0; no longer IC101.PA5/SPI1_SCK/ADC12_IN5
- net N$24: now also C103.2, IC101MCU.OSC_OUT, Q101.1; no longer C501.2, J509.4, R2.1
- net N$25: now also IC101MCU.PB1; no longer J509.3, R3.1
- net N$26: now also IC101MCU.PB2; no longer J509.2, R4.1
- net N$28: now also IC101MCU.PC0; no longer IC101.PB2/BOOT1
- net N$3: now also IC101MCU.PC15; no longer IC101.PB13/SPI2_SCK/USART3_CTS/TIM1_CH1N, R103.1
- net N$4: now also IC101MCU.PC14; no longer IC101.PA0/WKUP/USART2_CTS/ADC12_IN0/TIM2_CH1_ETR
- net N$42: now also IC101MCU.PB5; no longer D402.C, Q401.G, R401.2
- net N$43: now also IC101MCU.PB4; no longer IC401.EMIT, IC402.COL, R402.2
- net N$44: now also IC101MCU.PA6; no longer IC401.A, R403.1
- net N$45: now also D402.A, J405.4; no longer IC402.A, R404.1
- net N$5: now also IC101MCU.PC13; no longer IC101.PC13/TAMPERRTC
- net N$51: now also IC101MCU.PB14; no longer IC101.PB5/I2C1_SMBAL[TIM3_CH2/SPI1_MOSI]
- net N$57: now also IC101MCU.PA0-WKUP; no longer IC101.PC15/OSC32_OUT
- net N$6: now also IC101MCU.PC1; no longer C103.2, IC101.PD1/OSC_OUT, Q101.1
- net N$7: now also J409.3, J410.3, R405.1; no longer C102.1, IC101.PD0/OSC_IN, Q101.2
- net N$9: now also C301.2, IC306.RST; no longer IC301.TXD, R301.2
- net VBAT: now also IC101MCU.VBAT; no longer IC101.VBAT
- net VDD: now also C108.2, D402.C, IC101MCU.VDDA, IC101PWR.VDD@1, IC101PWR.VDD@2, IC101PWR.VDD@3, IC101PWR.VDD@4, IC306.VCC; no longer IC101.VDDA, IC101.VDD_1, IC101.VDD_2, IC101.VDD_3
Other:
- note added: "RELAY_ENABLE"
- note removed: "USART1_RXD"
- note removed: "USART1_TXD"
